Commit message: fix: set correct path for assets

File: src/nav2_gps_waypoint_follower_demo/urdf/gz_waffle.sdf.xacro (robot description, xacro)
@@ -30,5 +30,5 @@
           <geometry>
             <mesh>
-              <uri>package://nav2_minimal_tb3_sim/models/turtlebot3_model/meshes/waffle_base.dae</uri>
+              <uri>package://nav2_gps_waypoint_follower_demo/models/turtlebot3_model/meshes/waffle_base.dae</uri>
               <scale>0.001 0.001 0.001</scale>
             </mesh>
@@ -115,5 +115,5 @@
           <geometry>
             <mesh>
-              <uri>package://nav2_minimal_tb3_sim/models/turtlebot3_model/meshes/lds.dae</uri>
+              <uri>package://nav2_gps_waypoint_follower_demo/models/turtlebot3_model/meshes/lds.dae</uri>
               <scale>0.001 0.001 0.001</scale>
             </mesh>
@@ -199,5 +199,5 @@
           <geometry>
             <mesh>
-              <uri>package://nav2_minimal_tb3_sim/models/turtlebot3_model/meshes/tire.dae</uri>
+              <uri>package://nav2_gps_waypoint_follower_demo/models/turtlebot3_model/meshes/tire.dae</uri>
               <scale>0.001 0.001 0.001</scale>
             </mesh>
@@ -255,5 +255,5 @@
           <geometry>
             <mesh>
-              <uri>package://nav2_minimal_tb3_sim/models/turtlebot3_model/meshes/tire.dae</uri>
+              <uri>package://nav2_gps_waypoint_follower_demo/models/turtlebot3_model/meshes/tire.dae</uri>
               <scale>0.001 0.001 0.001</scale>
             </mesh>

File: src/nav2_gps_waypoint_follower_demo/urdf/gz_waffle_gps.sdf.xacro (robot description, xacro)
@@ -30,5 +30,5 @@
           <geometry>
             <mesh>
-              <uri>package://nav2_minimal_tb3_sim/models/turtlebot3_model/meshes/waffle_base.dae</uri>
+              <uri>package://nav2_gps_waypoint_follower_demo/models/turtlebot3_model/meshes/waffle_base.dae</uri>
               <scale>0.001 0.001 0.001</scale>
             </mesh>
@@ -141,5 +141,5 @@
           <geometry>
             <mesh>
-              <uri>package://nav2_minimal_tb3_sim/models/turtlebot3_model/meshes/lds.dae</uri>
+              <uri>package://nav2_gps_waypoint_follower_demo/models/turtlebot3_model/meshes/lds.dae</uri>
               <scale>0.001 0.001 0.001</scale>
             </mesh>
@@ -225,5 +225,5 @@
           <geometry>
             <mesh>
-              <uri>package://nav2_minimal_tb3_sim/models/turtlebot3_model/meshes/tire.dae</uri>
+              <uri>package://nav2_gps_waypoint_follower_demo/models/turtlebot3_model/meshes/tire.dae</uri>
               <scale>0.001 0.001 0.001</scale>
             </mesh>
@@ -281,5 +281,5 @@
           <geometry>
             <mesh>
-              <uri>package://nav2_minimal_tb3_sim/models/turtlebot3_model/meshes/tire.dae</uri>
+              <uri>package://nav2_gps_waypoint_follower_demo/models/turtlebot3_model/meshes/tire.dae</uri>
               <scale>0.001 0.001 0.001</scale>
             </mesh>

File: src/nav2_gps_waypoint_follower_demo/urdf/icreate/caster.urdf.xacro (robot description, xacro)
@@ -2,5 +2,5 @@
 <robot xmlns:xacro="http://ros.org/wiki/xacro">
 <xacro:macro name="caster" params="name parent_link *origin">
-  <xacro:include filename="$(find nav2_minimal_tb4_description)/urdf/icreate/common_properties.urdf.xacro"/>
+  <xacro:include filename="$(find nav2_gps_waypoint_follower_demo)/urdf/icreate/common_properties.urdf.xacro"/>
   <xacro:property name="radius" value="${1*cm2m}" />
   <xacro:property name="mass"   value="0.01"/>

File: src/nav2_gps_waypoint_follower_demo/urdf/icreate/create3.urdf.xacro (robot description, xacro)
@@ -1,9 +1,9 @@
 <?xml version="1.0" ?>
 <robot name="create3" xmlns:xacro="http://ros.org/wiki/xacro">
-  <xacro:include filename="$(find nav2_minimal_tb4_description)/urdf/icreate/bumper.urdf.xacro" />
-  <xacro:include filename="$(find nav2_minimal_tb4_description)/urdf/icreate/caster.urdf.xacro" />
-  <xacro:include filename="$(find nav2_minimal_tb4_description)/urdf/icreate/common_properties.urdf.xacro"/>
-  <xacro:include filename="$(find nav2_minimal_tb4_description)/urdf/icreate/sensors/imu.urdf.xacro" />
-  <xacro:include filename="$(find nav2_minimal_tb4_description)/urdf/icreate/wheel.urdf.xacro" />
+  <xacro:include filename="$(find nav2_gps_waypoint_follower_demo)/urdf/icreate/bumper.urdf.xacro" />
+  <xacro:include filename="$(find nav2_gps_waypoint_follower_demo)/urdf/icreate/caster.urdf.xacro" />
+  <xacro:include filename="$(find nav2_gps_waypoint_follower_demo)/urdf/icreate/common_properties.urdf.xacro"/>
+  <xacro:include filename="$(find nav2_gps_waypoint_follower_demo)/urdf/icreate/sensors/imu.urdf.xacro" />
+  <xacro:include filename="$(find nav2_gps_waypoint_follower_demo)/urdf/icreate/wheel.urdf.xacro" />
   <!-- Gazebo version -->
   <xacro:arg name="gazebo"                       default="ignition" />
@@ -33,5 +33,5 @@
       <origin xyz="0 0 ${body_z_offset + base_link_z_offset}" rpy="0 0 ${pi/2}"/>
       <geometry>
-        <mesh filename="package://nav2_minimal_tb4_description/meshes/body_visual.dae" />
+        <mesh filename="package://nav2_gps_waypoint_follower_demo/meshes/body_visual.dae" />
       </geometry>
     </visual>
@@ -53,6 +53,6 @@
       gazebo="$(arg gazebo)"
       namespace="$(arg namespace)"
-      visual_mesh="package://nav2_minimal_tb4_description/meshes/bumper_visual.dae"
-      collision_mesh="package://nav2_minimal_tb4_description/meshes/bumper_collision.dae">
+      visual_mesh="package://nav2_gps_waypoint_follower_demo/meshes/bumper_visual.dae"
+      collision_mesh="package://nav2_gps_waypoint_follower_demo/meshes/bumper_collision.dae">
     <origin xyz="0 0 ${bumper_offset_z  + base_link_z_offset}"/>
     <inertial>

File: src/nav2_gps_waypoint_follower_demo/urdf/sensors/camera_bracket.urdf.xacro (robot description, xacro)
@@ -1,5 +1,5 @@
 <?xml version="1.0"?>
 <robot xmlns:xacro="http://ros.org/wiki/xacro">
-<xacro:include filename="$(find nav2_minimal_tb4_description)/urdf/icreate/common_properties.urdf.xacro"/>
+<xacro:include filename="$(find nav2_gps_waypoint_follower_demo)/urdf/icreate/common_properties.urdf.xacro"/>
 <xacro:macro name="camera_bracket" params="name parent_link:=shell_link *origin">
   <xacro:property name="mass" value="0.033"/>
@@ -14,5 +14,5 @@
     <visual>
       <geometry>
-       <mesh filename="package://nav2_minimal_tb4_description/meshes/camera_bracket.dae" scale="1 1 1" />
+       <mesh filename="package://nav2_gps_waypoint_follower_demo/meshes/camera_bracket.dae" scale="1 1 1" />
       </geometry>
     </visual>

File: src/nav2_gps_waypoint_follower_demo/urdf/sensors/oakd.urdf.xacro (robot description, xacro)
@@ -2,5 +2,5 @@
 <robot xmlns:xacro="http://ros.org/wiki/xacro">
 <xacro:macro name="oakd" params="name:=oakd parent_link *origin model:=pro">
-  <xacro:include filename="$(find nav2_minimal_tb4_description)/urdf/icreate/common_properties.urdf.xacro"/>
+  <xacro:include filename="$(find nav2_gps_waypoint_follower_demo)/urdf/icreate/common_properties.urdf.xacro"/>
   <xacro:property name="mass"       value="0.061"/>
   <xacro:property name="baseline" value="0.075" />
@@ -22,5 +22,5 @@
     <visual>
       <geometry>
-        <mesh filename="package://nav2_minimal_tb4_description/meshes/${name}_${model}.dae" scale="1 1 1" />
+        <mesh filename="package://nav2_gps_waypoint_follower_demo/meshes/${name}_${model}.dae" scale="1 1 1" />
       </geometry>
     </visual>

File: src/nav2_gps_waypoint_follower_demo/urdf/sensors/rplidar.urdf.xacro (robot description, xacro)
@@ -2,5 +2,5 @@
 <robot xmlns:xacro="http://ros.org/wiki/xacro">
 <xacro:macro name="rplidar" params="name parent_link gazebo *origin">
-  <xacro:include filename="$(find nav2_minimal_tb4_description)/urdf/icreate/common_properties.urdf.xacro"/>
+  <xacro:include filename="$(find nav2_gps_waypoint_follower_demo)/urdf/icreate/common_properties.urdf.xacro"/>
   <xacro:property name="mass"       value="0.17"/>
   <xacro:property name="length_x"   value="${7.1*cm2m}" />
@@ -18,5 +18,5 @@
     <visual>
       <geometry>
-        <mesh filename="package://nav2_minimal_tb4_description/meshes/rplidar.dae" scale="1 1 1" />
+        <mesh filename="package://nav2_gps_waypoint_follower_demo/meshes/rplidar.dae" scale="1 1 1" />
       </geometry>
     </visual>

File: src/nav2_gps_waypoint_follower_demo/urdf/standard/tower_sensor_plate.urdf.xacro (robot description, xacro)
@@ -1,5 +1,5 @@
 <?xml version="1.0"?>
 <robot xmlns:xacro="http://ros.org/wiki/xacro">
-<xacro:include filename="$(find nav2_minimal_tb4_description)/urdf/icreate/common_properties.urdf.xacro"/>
+<xacro:include filename="$(find nav2_gps_waypoint_follower_demo)/urdf/icreate/common_properties.urdf.xacro"/>
 <xacro:macro name="tower_sensor_plate" params="name parent_link:=shell_link *origin">
   <xacro:property name="link_name" value="${name}"/>
@@ -14,5 +14,5 @@
     <visual>
       <geometry>
-       <mesh filename="package://nav2_minimal_tb4_description/meshes/tower_sensor_plate.dae" scale="1 1 1" />
+       <mesh filename="package://nav2_gps_waypoint_follower_demo/meshes/tower_sensor_plate.dae" scale="1 1 1" />
       </geometry>
     </visual>

File: src/nav2_gps_waypoint_follower_demo/urdf/standard/tower_standoff.urdf.xacro (robot description, xacro)
@@ -1,5 +1,5 @@
 <?xml version="1.0"?>
 <robot xmlns:xacro="http://ros.org/wiki/xacro">
-<xacro:include filename="$(find nav2_minimal_tb4_description)/urdf/icreate/common_properties.urdf.xacro"/>
+<xacro:include filename="$(find nav2_gps_waypoint_follower_demo)/urdf/icreate/common_properties.urdf.xacro"/>
 <xacro:macro name="tower_standoff" params="name parent_link:=shell_link *origin">
   <xacro:property name="link_name" value="${name}"/>
@@ -15,5 +15,5 @@
       <origin rpy="0 ${pi/2} 0"/>
       <geometry>
-       <mesh filename="package://nav2_minimal_tb4_description/meshes/tower_standoff.dae" scale="1 1 1" />
+       <mesh filename="package://nav2_gps_waypoint_follower_demo/meshes/tower_standoff.dae" scale="1 1 1" />
       </geometry>
     </visual>

File: src/nav2_gps_waypoint_follower_demo/urdf/standard/turtlebot4.urdf.xacro (robot description, xacro)
@@ -2,11 +2,11 @@
 <robot name="turtlebot4" xmlns:xacro="http://ros.org/wiki/xacro">
   <!-- Base create3 model -->
-  <xacro:include filename="$(find nav2_minimal_tb4_description)/urdf/icreate/create3.urdf.xacro" />
-  <xacro:include filename="$(find nav2_minimal_tb4_description)/urdf/sensors/rplidar.urdf.xacro" />
-  <xacro:include filename="$(find nav2_minimal_tb4_description)/urdf/sensors/oakd.urdf.xacro" />
-  <xacro:include filename="$(find nav2_minimal_tb4_description)/urdf/sensors/camera_bracket.urdf.xacro" />
-  <xacro:include filename="$(find nav2_minimal_tb4_description)/urdf/standard/tower_standoff.urdf.xacro" />
-  <xacro:include filename="$(find nav2_minimal_tb4_description)/urdf/standard/tower_sensor_plate.urdf.xacro" />
-  <xacro:include filename="$(find nav2_minimal_tb4_description)/urdf/standard/weight_block.urdf.xacro" />
+  <xacro:include filename="$(find nav2_gps_waypoint_follower_demo)/urdf/icreate/create3.urdf.xacro" />
+  <xacro:include filename="$(find nav2_gps_waypoint_follower_demo)/urdf/sensors/rplidar.urdf.xacro" />
+  <xacro:include filename="$(find nav2_gps_waypoint_follower_demo)/urdf/sensors/oakd.urdf.xacro" />
+  <xacro:include filename="$(find nav2_gps_waypoint_follower_demo)/urdf/sensors/camera_bracket.urdf.xacro" />
+  <xacro:include filename="$(find nav2_gps_waypoint_follower_demo)/urdf/standard/tower_standoff.urdf.xacro" />
+  <xacro:include filename="$(find nav2_gps_waypoint_follower_demo)/urdf/standard/tower_sensor_plate.urdf.xacro" />
+  <xacro:include filename="$(find nav2_gps_waypoint_follower_demo)/urdf/standard/weight_block.urdf.xacro" />
   <!-- Mechanical properties -->
   <xacro:property name="shell_z_offset"                value="${3*cm2m}" />
@@ -62,10 +62,10 @@
       <origin xyz="0 0 0" rpy="${pi/2} 0 ${pi/2}"/>
       <geometry>
-        <mesh filename="package://nav2_minimal_tb4_description/meshes/shell.dae" scale="1 1 1" />
+        <mesh filename="package://nav2_gps_waypoint_follower_demo/meshes/shell.dae" scale="1 1 1" />
       </geometry>
     </visual>
     <collision name="shell_collision">
       <geometry>
-        <mesh filename="package://nav2_minimal_tb4_description/meshes/shell_collision.dae" scale="1 1 1" />
+        <mesh filename="package://nav2_gps_waypoint_follower_demo/meshes/shell_collision.dae" scale="1 1 1" />
       </geometry>
     </collision>

File: src/nav2_gps_waypoint_follower_demo/urdf/standard/weight_block.urdf.xacro (robot description, xacro)
@@ -1,5 +1,5 @@
 <?xml version="1.0"?>
 <robot xmlns:xacro="http://ros.org/wiki/xacro">
-<xacro:include filename="$(find nav2_minimal_tb4_description)/urdf/icreate/common_properties.urdf.xacro"/>
+<xacro:include filename="$(find nav2_gps_waypoint_follower_demo)/urdf/icreate/common_properties.urdf.xacro"/>
 <xacro:macro name="weight_block" params="name parent_link:=base_link *origin">
   <xacro:property name="link_name" value="${name}"/>
@@ -14,5 +14,5 @@
     <visual>
       <geometry>
-       <mesh filename="package://nav2_minimal_tb4_description/meshes/weight_block.dae" scale="1 1 1" />
+       <mesh filename="package://nav2_gps_waypoint_follower_demo/meshes/weight_block.dae" scale="1 1 1" />
       </geometry>
     </visual>

File: src/nav2_gps_waypoint_follower_demo/urdf/turtlebot3_waffle.urdf (robot description, URDF)
Before this commit: robot turtlebot3_waffle, 13 links, 12 joints
Links:
- link base_link: geometry collision box size=0.266 0.266 0.094; visual mesh filename=package://nav2_gps_waypoint_follower_demo/models/turtlebot3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 scale=0.001 0.001 0.001
- link base_scan: geometry collision cylinder length=0.0315 radius=0.055; visual mesh filename=package://nav2_gps_waypoint_follower_demo/models/turtlebot3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 scale=0.001 0.001 0.001
- link camera_link: geometry collision box size=0.012 0.132 0.020; visual mesh filename=package://nav2_gps_waypoint_follower_demo/models/turtlebot3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
- link wheel_left_link: geometry collision cylinder length=0.018 radius=0.033; visual mesh filename=package://nav2_gps_waypoint_follower_demo/models/turtlebot3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 scale=0.001 0.001 0.001
- link wheel_right_link: geometry collision cylinder length=0.018 radius=0.033; visual mesh filename=package://nav2_gps_waypoint_follower_demo/models/turtlebot3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 scale=0.001 0.001 0.001

File: src/nav2_gps_waypoint_follower_demo/urdf/turtlebot3_waffle_gps.urdf (robot description, URDF)
Before this commit: robot turtlebot3_waffle, 14 links, 13 joints
Links:
- link base_link: geometry collision box size=0.266 0.266 0.094; visual mesh filename=package://nav2_gps_waypoint_follower_demo/models/turtlebot3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 scale=0.001 0.001 0.001
- link base_scan: geometry collision cylinder length=0.0315 radius=0.055; visual mesh filename=package://nav2_gps_waypoint_follower_demo/models/turtlebot3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 scale=0.001 0.001 0.001
- link camera_link: geometry collision box size=0.012 0.132 0.020; visual mesh filename=package://nav2_gps_waypoint_follower_demo/models/turtlebot3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
- link wheel_left_link: geometry collision cylinder length=0.018 radius=0.033; visual mesh filename=package://nav2_gps_waypoint_follower_demo/models/turtlebot3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 scale=0.001 0.001 0.001
- link wheel_right_link: geometry collision cylinder length=0.018 radius=0.033; visual mesh filename=package://nav2_gps_waypoint_follower_demo/models/turtlebot3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 scale=0.001 0.001 0.001
